Commit message: dealing with joint4

File: franka_fr3_moveit_config/srdf/group_definition.xacro (robot description, xacro)
@@ -9,5 +9,5 @@
       <joint name="${arm_id}_joint2" value="${-pi/4}"/>
       <joint name="${arm_id}_joint3" value="0"/>
-      <joint name="${arm_id}_joint4" value="${-3*pi/4}"/>
+      <joint name="${arm_id}_joint4" value="0"/>
       <joint name="${arm_id}_joint5" value="0"/>
       <joint name="${arm_id}_joint6" value="${pi/2}"/>

Commit message: link5

File: franka_fr3_moveit_config/srdf/group_definition.xacro (robot description, xacro)
@@ -10,5 +10,5 @@
       <joint name="${arm_id}_joint3" value="0"/>
       <joint name="${arm_id}_joint4" value="0"/>
-      <joint name="${arm_id}_joint5" value="0"/>
+      <joint name="${arm_id}_joint5" value="${pi/2}"/>
       <joint name="${arm_id}_joint6" value="${pi/2}"/>
       <joint name="${arm_id}_joint7" value="${pi/4}"/>

Commit message: some further link4 and link5 fixes

File: franka_fr3_moveit_config/srdf/group_definition.xacro (robot description, xacro)
@@ -7,7 +7,7 @@
     <group_state name="ready" group="${group_name}">
       <joint name="${arm_id}_joint1" value="0"/>
-      <joint name="${arm_id}_joint2" value="${-pi/4}"/>
+      <joint name="${arm_id}_joint2" value="0"/>
       <joint name="${arm_id}_joint3" value="0"/>
-      <joint name="${arm_id}_joint4" value="${-3*pi/4}"/>
+      <joint name="${arm_id}_joint4" value="0"/>
       <joint name="${arm_id}_joint5" value="0"/>
       <joint name="${arm_id}_joint6" value="${pi/2}"/>
@@ -18,5 +18,5 @@
       <joint name="${arm_id}_joint2" value="0"/>
       <joint name="${arm_id}_joint3" value="0"/>
-      <joint name="${arm_id}_joint4" value="-0.1"/>
+      <joint name="${arm_id}_joint4" value="0"/>
       <joint name="${arm_id}_joint5" value="0"/>
       <joint name="${arm_id}_joint6" value="${pi/2}"/>
